Commit message: Нормально настроен гриппер

File: iiwa_ros2/iiwa_description/ros2_control/iiwa.r2c_hardware.xacro (robot description, xacro)
@@ -136,4 +136,36 @@
                 </state_interface>
             </joint>
+            <joint name="${prefix}joint_finger_1">
+                <command_interface name="${command_interface}" />
+                    <xacro:if value="${command_interface == 'position'}">
+                        <param name="min">0.0</param>
+                        <param name="max">0.033</param>
+                    </xacro:if>
+                <state_interface name="position">
+                    <param name="initial_value">${initial_positions['joint_finger_1']}</param>
+                </state_interface>
+                <state_interface name="velocity">
+                    <param name="initial_value">0.0</param>
+                </state_interface>
+                <state_interface name="effort">
+                    <param name="initial_value">0.0</param>
+                </state_interface>
+            </joint>
+            <joint name="${prefix}joint_finger_2">
+                <command_interface name="${command_interface}" />
+                    <xacro:if value="${command_interface == 'position'}">
+                        <param name="min">-0.033</param>
+                        <param name="max">0.0</param>
+                    </xacro:if>
+                <state_interface name="position">
+                    <param name="initial_value">${initial_positions['joint_finger_2']}</param>
+                </state_interface>
+                <state_interface name="velocity">
+                    <param name="initial_value">0.0</param>
+                </state_interface>
+                <state_interface name="effort">
+                    <param name="initial_value">0.0</param>
+                </state_interface>
+            </joint>
             <sensor name="${prefix}external_torque_sensor">
                 <state_interface name="external_torque.joint_a1">
@@ -156,4 +188,10 @@
                 </state_interface>
                 <state_interface name="external_torque.joint_a7">
+                    <param name="initial_value">0.0</param>
+                </state_interface>
+                <state_interface name="external_torque.joint_finger_1">
+                    <param name="initial_value">0.0</param>
+                </state_interface>
+                <state_interface name="external_torque.joint_finger_2">
                     <param name="initial_value">0.0</param>
                 </state_interface>

File: iiwa_ros2/iiwa_description/ros2_control/iiwa.r2c_hw_ds.xacro (robot description, xacro)
@@ -58,4 +58,18 @@
                 <state_interface name="position"/>
             </joint>
+            <joint name="joint_finger_1">
+                <param name="initial_position">${initial_positions['joint_finger_1']}</param>
+                <command_interface name="position" />
+                    <param name="min">0.0</param>
+                    <param name="max">0.033</param>
+                <state_interface name="position"/>
+            </joint>
+            <joint name="joint_finger_2">
+                <param name="initial_position">${initial_positions['joint_finger_2']}</param>
+                <command_interface name="position" />
+                    <param name="min">-0.033</param>
+                    <param name="max">0.0</param>
+                <state_interface name="position"/>
+            </joint>
         </ros2_control>
     </xacro:macro>

File: iiwa_ros2/iiwa_description/srdf/iiwa_macro.srdf.xacro (robot description, xacro)
@@ -3,5 +3,5 @@
   <xacro:macro name="iiwa_srdf" params="name prefix">
     <group name="${prefix}${name}_arm">
-        <chain base_link="${prefix}iiwa_base" tip_link="${prefix}joint_finger_1" />
+        <chain base_link="${prefix}iiwa_base" tip_link="${prefix}tool0" />
     </group>
     <group_state name="ready" group="${prefix}${name}_arm">
@@ -13,5 +13,6 @@
         <joint name="${prefix}joint_a6" value="1.571"/>
         <joint name="${prefix}joint_a7" value="0.785"/>
-        <joint name="${prefix}joint_a7-tool0" value="0"/>
+        <joint name="${prefix}joint_finger_1" value="0"/>
+        <joint name="${prefix}joint_finger_2" value="0"/>
     </group_state>
     <virtual_joint child_link="${prefix}iiwa_base" name="virtual_joint" parent_frame="world" type="floating"/>
@@ -32,4 +33,5 @@
     <disable_collisions link1="${prefix}link_1" link2="${prefix}tool0" reason="Never" />
     <disable_collisions link1="${prefix}link_1" link2="${prefix}link_gripper_finger_1" reason="Never" />
+    <disable_collisions link1="${prefix}link_1" link2="${prefix}link_gripper_finger_2" reason="Never" />
     <disable_collisions link1="${prefix}link_2" link2="${prefix}link_3" reason="Adjacent" />
     <disable_collisions link1="${prefix}link_2" link2="${prefix}link_4" reason="Never" />
@@ -39,4 +41,5 @@
     <disable_collisions link1="${prefix}link_2" link2="${prefix}tool0" reason="Never" />
     <disable_collisions link1="${prefix}link_2" link2="${prefix}link_gripper_finger_1" reason="Never" />
+    <disable_collisions link1="${prefix}link_2" link2="${prefix}link_gripper_finger_2" reason="Never" />
     <disable_collisions link1="${prefix}link_3" link2="${prefix}link_4" reason="Adjacent" />
     <disable_collisions link1="${prefix}link_3" link2="${prefix}link_5" reason="Never" />
@@ -45,4 +48,5 @@
     <disable_collisions link1="${prefix}link_3" link2="${prefix}tool0" reason="Never" />
     <disable_collisions link1="${prefix}link_3" link2="${prefix}link_gripper_finger_1" reason="Never" />
+    <disable_collisions link1="${prefix}link_3" link2="${prefix}link_gripper_finger_2" reason="Never" />
     <disable_collisions link1="${prefix}link_4" link2="${prefix}link_5" reason="Adjacent" />
     <disable_collisions link1="${prefix}link_4" link2="${prefix}link_6" reason="Never" />
@@ -50,14 +54,21 @@
     <disable_collisions link1="${prefix}link_4" link2="${prefix}tool0" reason="Never" />
     <disable_collisions link1="${prefix}link_4" link2="${prefix}link_gripper_finger_1" reason="Never" />
+    <disable_collisions link1="${prefix}link_4" link2="${prefix}link_gripper_finger_2" reason="Never" />
     <disable_collisions link1="${prefix}link_5" link2="${prefix}link_6" reason="Adjacent" />
     <disable_collisions link1="${prefix}link_5" link2="${prefix}link_7" reason="Never" />
     <disable_collisions link1="${prefix}link_5" link2="${prefix}tool0" reason="Never" />
     <disable_collisions link1="${prefix}link_5" link2="${prefix}link_gripper_finger_1" reason="Never" />
+    <disable_collisions link1="${prefix}link_5" link2="${prefix}link_gripper_finger_2" reason="Never" />
     <disable_collisions link1="${prefix}link_6" link2="${prefix}link_7" reason="Adjacent" />
     <disable_collisions link1="${prefix}link_6" link2="${prefix}tool0" reason="Never" />
     <disable_collisions link1="${prefix}link_6" link2="${prefix}link_gripper_finger_1" reason="Never" />
+    <disable_collisions link1="${prefix}link_6" link2="${prefix}link_gripper_finger_2" reason="Never" />
     <disable_collisions link1="${prefix}link_7" link2="${prefix}tool0" reason="Adjacent" />
     <disable_collisions link1="${prefix}link_7" link2="${prefix}link_gripper_finger_1" reason="Never" />
+    <disable_collisions link1="${prefix}link_7" link2="${prefix}link_gripper_finger_2" reason="Never" />
     <disable_collisions link1="${prefix}tool0" link2="${prefix}link_gripper_finger_1" reason="Adjacent" />
+    <disable_collisions link1="${prefix}link_gripper_finger_1" link2="${prefix}link_gripper_finger_2" reason="Never" />
+    <disable_collisions link1="${prefix}tool0" link2="${prefix}link_gripper_finger_2" reason="Adjacent" />
+    <disable_collisions link1="${prefix}link_gripper_finger_2" link2="${prefix}link_gripper_finger_1" reason="Never" />
   </xacro:macro>
 </robot>

File: iiwa_ros2/iiwa_description/urdf/iiwa.urdf.xacro (robot description, xacro)
@@ -284,13 +284,17 @@
       <axis xyz="0 0 0"/>
   </joint>
-  <joint name="${prefix}joint_finger_1" type="fixed">
-      <origin rpy="0.0 0 0" xyz="0 0 0"/>
-      <parent link="${prefix}tool0"/>
-      <child link="${prefix}link_gripper_finger_1"/>
-  </joint>
-  <joint name="${prefix}joint_finger_2" type="fixed">
-      <origin rpy="0.0 0 0" xyz="0 0 0"/>
-      <parent link="${prefix}tool0"/>
-      <child link="${prefix}link_gripper_finger_2"/>
+  <joint name="${prefix}joint_finger_1" type="prismatic">
+    <origin xyz="0 0 0" rpy="0 0 0"/>
+    <parent link="${prefix}tool0"/>
+    <child link="${prefix}link_gripper_finger_1"/>
+    <axis xyz="0 1 0"/>
+    <limit lower="0" upper="0.033" velocity="100" effort="100"/>
+  </joint>
+  <joint name="${prefix}joint_finger_2" type="prismatic">
+    <origin xyz="0 0 0" rpy="0 0 0"/>
+    <parent link="${prefix}tool0"/>
+    <child link="${prefix}link_gripper_finger_2"/>
+    <axis xyz="0 1 0"/>
+    <limit lower="-0.033" upper="0" velocity="100" effort="100"/>
   </joint>
   </xacro:macro>
